File: Dashcam_HAT.sch (EAGLE design)
At the start: 73 parts, among them J1 RJ45-8PTH, J2 JST_VERTICAL, J3 PIN20X2, J5 M4, J7 6_PIN_SMD, Q1 MMBT2222, Q2 MMBT2222, U1 STN1110, U2 MCP2551, U3 TS30011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

Commit message: Added missing attributes for TL331 comparator
Parts:
- U7: DIGIKEY_PN (none) -> 296-10168-1-ND; MANUFACTURER (none) -> Texas Instruments; MFG_PN (none) -> TL331IDBVR
Changed lines of the file:
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@@
 <part name="P+13" library="SparkFun" deviceset="VCC" device="" value="VBATT"/>
 <part name="GND22" library="SparkFun" deviceset="GND" device=""/>
-<part name="U7" library="linear" deviceset="TL331" device=""/>
+<part name="U7" library="linear" deviceset="TL331" device="">
+<attribute name="DIGIKEY_PN" value="296-10168-1-ND"/>
+<attribute name="MANUFACTURER" value="Texas Instruments"/>
+<attribute name="MFG_PN" value="TL331IDBVR"/>
+</part>
 <part name="VBAT" library="SparkFun" deviceset="VCC" device="" value="VBATT"/>
 <part name="Q2" library="SparkFun" deviceset="TRANSISTOR_NPN" device="SOT23-3" value="MMBT2222">
@@
 <instance part="P+13" gate="1" x="330.2" y="223.52"/>
 <instance part="GND22" gate="1" x="330.2" y="195.58" rot="MR0"/>
-<instance part="U7" gate="G$1" x="330.2" y="208.28"/>
+<instance part="U7" gate="G$1" x="330.2" y="208.28">
+<attribute name="DIGIKEY_PN" x="330.2" y="208.28" size="1.778" layer="96" display="off"/>
+<attribute name="MANUFACTURER" x="330.2" y="208.28" size="1.778" layer="96" display="off"/>
+<attribute name="MFG_PN" x="330.2" y="208.28" size="1.778" layer="96" display="off"/>
+</instance>
 <instance part="VBAT" gate="1" x="101.6" y="223.52"/>
 <instance part="Q2" gate="G$1" x="342.9" y="154.94" smashed="yes">

Commit message: Updated part identifiers
Parts:
- added J4: M4, Jason_Connector:M4
- renumbered C11 to C3
Connections:
- new net UART1_RX: J3.10
- new net UART1_TX: J3.8
Other:
- moved on the sheet: C2, R6, R61, S1

Commit message: Tweaked layout a bit and added more bypass caps
Parts:
- removed C40: 10uF, SparkFun-Capacitors:CAP1206
- added C25: 0.1uF, SparkFun:CAP0402-CAP
- added C44, C45: 10uF, SparkFun-Capacitors:CAP1206
- added D5: SMAJ16A, Jason_Library_1:DIODESMA
- J4: value M4 -> M30.1"_LOCK; device Jason_Connector:M4 -> Jason_Connector:M30.1"_LOCK
Connections:
- net N$16 renamed VSW
- net N$19 renamed BST
- net 5V: now also C43.1, C44.1; no longer C41.1
- net GND: now also C25.1, C44.2, C45.2, D5.A, J4.3; no longer C40.2
- net UART1_RX: now also J4.1
- net UART1_TX: now also J4.2
- net VBATT: now also C25.2, C41.1, C45.1, D5.C; no longer C40.1, C43.1
Other:
- moved on the sheet: C24, C41, C42, C43, D3, L1, R70, U3
